Commit message: anubis_v3 with mass refer from mobile aloha

File: anubis/urdf/anubis_v3.urdf (robot description, URDF)
Before this commit: robot anubis, 24 links, 23 joints
Links:
- link base_link: mass None -> 132.3898489950015
- link ee_link1: mass None -> 0.0062357399313257
- link ee_link2: mass None -> 0.0062357399313257
- link gripper2_base_link: mass None -> 0.62357399313257
- link gripper_base_link: mass None -> 0.62357399313257
- link link11: mass None -> 0.0608351104988555
- link link12: mass None -> 1.0733279014126
- link link13: mass None -> 0.499404738025019
- link link14: mass None -> 0.0809712553169999
- link link15: mass None -> 0.602357399313257
- link link21: mass None -> 0.0608351104988555
- link link22: mass None -> 1.0733279014126
- link link23: mass None -> 0.499404738025019
- link link24: mass None -> 0.0809712553169999
- link link25: mass None -> 0.602357399313257
