Commit message: fix mesh naming and config

File: eigenbot/eigenbot/source/eigenbot/eigenbot/assets/eigenbot/urdf/eigenbot_hexapod.urdf (robot description, URDF)
Before this commit: robot modular_robot_compiled, 50 links, 49 joints
Links:
- link bendy_input_M10_S10: geometry collision mesh filename=../meshes/Bendy_In.STL scale=1 1 1; visual mesh filename=../meshes/Bendy_In.STL scale=1 1 1
- link bendy_input_M11_S11: geometry collision mesh filename=../meshes/Bendy_In.STL scale=1 1 1; visual mesh filename=../meshes/Bendy_In.STL scale=1 1 1
- link bendy_input_M12_S12: geometry collision mesh filename=../meshes/Bendy_In.STL scale=1 1 1; visual mesh filename=../meshes/Bendy_In.STL scale=1 1 1
- link bendy_input_M13_S13: geometry collision mesh filename=../meshes/Bendy_In.STL scale=1 1 1; visual mesh filename=../meshes/Bendy_In.STL scale=1 1 1
- link bendy_input_M14_S14: geometry collision mesh filename=../meshes/Bendy_In.STL scale=1 1 1; visual mesh filename=../meshes/Bendy_In.STL scale=1 1 1
- link bendy_input_M15_S15: geometry collision mesh filename=../meshes/Bendy_In.STL scale=1 1 1; visual mesh filename=../meshes/Bendy_In.STL scale=1 1 1
- link bendy_input_M16_S16: geometry collision mesh filename=../meshes/Bendy_In.STL scale=1 1 1; visual mesh filename=../meshes/Bendy_In.STL scale=1 1 1
- link bendy_input_M17_S17: geometry collision mesh filename=../meshes/Bendy_In.STL scale=1 1 1; visual mesh filename=../meshes/Bendy_In.STL scale=1 1 1
- link bendy_input_M18_S18: geometry collision mesh filename=../meshes/Bendy_In.STL scale=1 1 1; visual mesh filename=../meshes/Bendy_In.STL scale=1 1 1
- link bendy_input_M1_S1: geometry collision mesh filename=../meshes/Bendy_In.STL scale=1 1 1; visual mesh filename=../meshes/Bendy_In.STL scale=1 1 1
- link bendy_input_M2_S2: geometry collision mesh filename=../meshes/Bendy_In.STL scale=1 1 1; visual mesh filename=../meshes/Bendy_In.STL scale=1 1 1
- link bendy_input_M3_S3: geometry collision mesh filename=../meshes/Bendy_In.STL scale=1 1 1; visual mesh filename=../meshes/Bendy_In.STL scale=1 1 1
- link bendy_input_M4_S4: geometry collision mesh filename=../meshes/Bendy_In.STL scale=1 1 1; visual mesh filename=../meshes/Bendy_In.STL scale=1 1 1
- link bendy_input_M5_S5: geometry collision mesh filename=../meshes/Bendy_In.STL scale=1 1 1; visual mesh filename=../meshes/Bendy_In.STL scale=1 1 1
- link bendy_input_M6_S6: geometry collision mesh filename=../meshes/Bendy_In.STL scale=1 1 1; visual mesh filename=../meshes/Bendy_In.STL scale=1 1 1
- link bendy_input_M7_S7: geometry collision mesh filename=../meshes/Bendy_In.STL scale=1 1 1; visual mesh filename=../meshes/Bendy_In.STL scale=1 1 1
- link bendy_input_M8_S8: geometry collision mesh filename=../meshes/Bendy_In.STL scale=1 1 1; visual mesh filename=../meshes/Bendy_In.STL scale=1 1 1
- link bendy_input_M9_S9: geometry collision mesh filename=../meshes/Bendy_In.STL scale=1 1 1; visual mesh filename=../meshes/Bendy_In.STL scale=1 1 1
- link bendy_output_M10_S10: geometry collision mesh filename=../meshes/Bendy_Out.STL scale=1 1 1; visual mesh filename=../meshes/Bendy_Out.STL scale=1 1 1
- link bendy_output_M11_S11: geometry collision mesh filename=../meshes/Bendy_Out.STL scale=1 1 1; visual mesh filename=../meshes/Bendy_Out.STL scale=1 1 1
- link bendy_output_M12_S12: geometry collision mesh filename=../meshes/Bendy_Out.STL scale=1 1 1; visual mesh filename=../meshes/Bendy_Out.STL scale=1 1 1
- link bendy_output_M13_S13: geometry collision mesh filename=../meshes/Bendy_Out.STL scale=1 1 1; visual mesh filename=../meshes/Bendy_Out.STL scale=1 1 1
- link bendy_output_M14_S14: geometry collision mesh filename=../meshes/Bendy_Out.STL scale=1 1 1; visual mesh filename=../meshes/Bendy_Out.STL scale=1 1 1
- link bendy_output_M15_S15: geometry collision mesh filename=../meshes/Bendy_Out.STL scale=1 1 1; visual mesh filename=../meshes/Bendy_Out.STL scale=1 1 1
- link bendy_output_M16_S16: geometry collision mesh filename=../meshes/Bendy_Out.STL scale=1 1 1; visual mesh filename=../meshes/Bendy_Out.STL scale=1 1 1
- link bendy_output_M17_S17: geometry collision mesh filename=../meshes/Bendy_Out.STL scale=1 1 1; visual mesh filename=../meshes/Bendy_Out.STL scale=1 1 1
- link bendy_output_M18_S18: geometry collision mesh filename=../meshes/Bendy_Out.STL scale=1 1 1; visual mesh filename=../meshes/Bendy_Out.STL scale=1 1 1
- link bendy_output_M1_S1: geometry collision mesh filename=../meshes/Bendy_Out.STL scale=1 1 1; visual mesh filename=../meshes/Bendy_Out.STL scale=1 1 1
- link bendy_output_M2_S2: geometry collision mesh filename=../meshes/Bendy_Out.STL scale=1 1 1; visual mesh filename=../meshes/Bendy_Out.STL scale=1 1 1
- link bendy_output_M3_S3: geometry collision mesh filename=../meshes/Bendy_Out.STL scale=1 1 1; visual mesh filename=../meshes/Bendy_Out.STL scale=1 1 1
- link bendy_output_M4_S4: geometry collision mesh filename=../meshes/Bendy_Out.STL scale=1 1 1; visual mesh filename=../meshes/Bendy_Out.STL scale=1 1 1
- link bendy_output_M5_S5: geometry collision mesh filename=../meshes/Bendy_Out.STL scale=1 1 1; visual mesh filename=../meshes/Bendy_Out.STL scale=1 1 1
- link bendy_output_M6_S6: geometry collision mesh filename=../meshes/Bendy_Out.STL scale=1 1 1; visual mesh filename=../meshes/Bendy_Out.STL scale=1 1 1
- link bendy_output_M7_S7: geometry collision mesh filename=../meshes/Bendy_Out.STL scale=1 1 1; visual mesh filename=../meshes/Bendy_Out.STL scale=1 1 1
- link bendy_output_M8_S8: geometry collision mesh filename=../meshes/Bendy_Out.STL scale=1 1 1; visual mesh filename=../meshes/Bendy_Out.STL scale=1 1 1
- link bendy_output_M9_S9: geometry collision mesh filename=../meshes/Bendy_Out.STL scale=1 1 1; visual mesh filename=../meshes/Bendy_Out.STL scale=1 1 1

Commit message: filename changes

File: eigenbot/eigenbot/source/eigenbot/eigenbot/assets/eigenbot/urdf/eigenbot_hexapod.urdf (robot description, URDF)
Before this commit: robot modular_robot_compiled, 50 links, 49 joints
Links:
- link bendy_input_M10_S10: geometry collision mesh filename=../meshes/BendyIn.STL scale=1 1 1; visual mesh filename=../meshes/BendyIn.STL scale=1 1 1
- link bendy_input_M11_S11: geometry collision mesh filename=../meshes/BendyIn.STL scale=1 1 1; visual mesh filename=../meshes/BendyIn.STL scale=1 1 1
- link bendy_input_M12_S12: geometry collision mesh filename=../meshes/BendyIn.STL scale=1 1 1; visual mesh filename=../meshes/BendyIn.STL scale=1 1 1
- link bendy_input_M13_S13: geometry collision mesh filename=../meshes/BendyIn.STL scale=1 1 1; visual mesh filename=../meshes/BendyIn.STL scale=1 1 1
- link bendy_input_M14_S14: geometry collision mesh filename=../meshes/BendyIn.STL scale=1 1 1; visual mesh filename=../meshes/BendyIn.STL scale=1 1 1
- link bendy_input_M15_S15: geometry collision mesh filename=../meshes/BendyIn.STL scale=1 1 1; visual mesh filename=../meshes/BendyIn.STL scale=1 1 1
- link bendy_input_M16_S16: geometry collision mesh filename=../meshes/BendyIn.STL scale=1 1 1; visual mesh filename=../meshes/BendyIn.STL scale=1 1 1
- link bendy_input_M17_S17: geometry collision mesh filename=../meshes/BendyIn.STL scale=1 1 1; visual mesh filename=../meshes/BendyIn.STL scale=1 1 1
- link bendy_input_M18_S18: geometry collision mesh filename=../meshes/BendyIn.STL scale=1 1 1; visual mesh filename=../meshes/BendyIn.STL scale=1 1 1
- link bendy_input_M1_S1: geometry collision mesh filename=../meshes/BendyIn.STL scale=1 1 1; visual mesh filename=../meshes/BendyIn.STL scale=1 1 1
- link bendy_input_M2_S2: geometry collision mesh filename=../meshes/BendyIn.STL scale=1 1 1; visual mesh filename=../meshes/BendyIn.STL scale=1 1 1
- link bendy_input_M3_S3: geometry collision mesh filename=../meshes/BendyIn.STL scale=1 1 1; visual mesh filename=../meshes/BendyIn.STL scale=1 1 1
- link bendy_input_M4_S4: geometry collision mesh filename=../meshes/BendyIn.STL scale=1 1 1; visual mesh filename=../meshes/BendyIn.STL scale=1 1 1
- link bendy_input_M5_S5: geometry collision mesh filename=../meshes/BendyIn.STL scale=1 1 1; visual mesh filename=../meshes/BendyIn.STL scale=1 1 1
- link bendy_input_M6_S6: geometry collision mesh filename=../meshes/BendyIn.STL scale=1 1 1; visual mesh filename=../meshes/BendyIn.STL scale=1 1 1
- link bendy_input_M7_S7: geometry collision mesh filename=../meshes/BendyIn.STL scale=1 1 1; visual mesh filename=../meshes/BendyIn.STL scale=1 1 1
- link bendy_input_M8_S8: geometry collision mesh filename=../meshes/BendyIn.STL scale=1 1 1; visual mesh filename=../meshes/BendyIn.STL scale=1 1 1
- link bendy_input_M9_S9: geometry collision mesh filename=../meshes/BendyIn.STL scale=1 1 1; visual mesh filename=../meshes/BendyIn.STL scale=1 1 1
- link bendy_output_M10_S10: geometry collision mesh filename=../meshes/BendyOut.STL scale=1 1 1; visual mesh filename=../meshes/BendyOut.STL scale=1 1 1
- link bendy_output_M11_S11: geometry collision mesh filename=../meshes/BendyOut.STL scale=1 1 1; visual mesh filename=../meshes/BendyOut.STL scale=1 1 1
- link bendy_output_M12_S12: geometry collision mesh filename=../meshes/BendyOut.STL scale=1 1 1; visual mesh filename=../meshes/BendyOut.STL scale=1 1 1
- link bendy_output_M13_S13: geometry collision mesh filename=../meshes/BendyOut.STL scale=1 1 1; visual mesh filename=../meshes/BendyOut.STL scale=1 1 1
- link bendy_output_M14_S14: geometry collision mesh filename=../meshes/BendyOut.STL scale=1 1 1; visual mesh filename=../meshes/BendyOut.STL scale=1 1 1
- link bendy_output_M15_S15: geometry collision mesh filename=../meshes/BendyOut.STL scale=1 1 1; visual mesh filename=../meshes/BendyOut.STL scale=1 1 1
- link bendy_output_M16_S16: geometry collision mesh filename=../meshes/BendyOut.STL scale=1 1 1; visual mesh filename=../meshes/BendyOut.STL scale=1 1 1
- link bendy_output_M17_S17: geometry collision mesh filename=../meshes/BendyOut.STL scale=1 1 1; visual mesh filename=../meshes/BendyOut.STL scale=1 1 1
- link bendy_output_M18_S18: geometry collision mesh filename=../meshes/BendyOut.STL scale=1 1 1; visual mesh filename=../meshes/BendyOut.STL scale=1 1 1
- link bendy_output_M1_S1: geometry collision mesh filename=../meshes/BendyOut.STL scale=1 1 1; visual mesh filename=../meshes/BendyOut.STL scale=1 1 1
- link bendy_output_M2_S2: geometry collision mesh filename=../meshes/BendyOut.STL scale=1 1 1; visual mesh filename=../meshes/BendyOut.STL scale=1 1 1
- link bendy_output_M3_S3: geometry collision mesh filename=../meshes/BendyOut.STL scale=1 1 1; visual mesh filename=../meshes/BendyOut.STL scale=1 1 1
- link bendy_output_M4_S4: geometry collision mesh filename=../meshes/BendyOut.STL scale=1 1 1; visual mesh filename=../meshes/BendyOut.STL scale=1 1 1
- link bendy_output_M5_S5: geometry collision mesh filename=../meshes/BendyOut.STL scale=1 1 1; visual mesh filename=../meshes/BendyOut.STL scale=1 1 1
- link bendy_output_M6_S6: geometry collision mesh filename=../meshes/BendyOut.STL scale=1 1 1; visual mesh filename=../meshes/BendyOut.STL scale=1 1 1
- link bendy_output_M7_S7: geometry collision mesh filename=../meshes/BendyOut.STL scale=1 1 1; visual mesh filename=../meshes/BendyOut.STL scale=1 1 1
- link bendy_output_M8_S8: geometry collision mesh filename=../meshes/BendyOut.STL scale=1 1 1; visual mesh filename=../meshes/BendyOut.STL scale=1 1 1
- link bendy_output_M9_S9: geometry collision mesh filename=../meshes/BendyOut.STL scale=1 1 1; visual mesh filename=../meshes/BendyOut.STL scale=1 1 1

Commit message: add rigidbody for usdz

File: eigenbot/eigenbot/source/eigenbot/eigenbot/assets/eigenbot/urdf/eigenbot_hexapod.urdf (robot description, URDF)
Before this commit: robot modular_robot_compiled, 50 links, 49 joints
Links:
- link bendy_input_M10_S10: geometry collision mesh filename=../meshes/bendyin.stl scale=1 1 1; visual mesh filename=../meshes/bendyin.stl scale=1 1 1
- link bendy_input_M11_S11: geometry collision mesh filename=../meshes/bendyin.stl scale=1 1 1; visual mesh filename=../meshes/bendyin.stl scale=1 1 1
- link bendy_input_M12_S12: geometry collision mesh filename=../meshes/bendyin.stl scale=1 1 1; visual mesh filename=../meshes/bendyin.stl scale=1 1 1
- link bendy_input_M13_S13: geometry collision mesh filename=../meshes/bendyin.stl scale=1 1 1; visual mesh filename=../meshes/bendyin.stl scale=1 1 1
- link bendy_input_M14_S14: geometry collision mesh filename=../meshes/bendyin.stl scale=1 1 1; visual mesh filename=../meshes/bendyin.stl scale=1 1 1
- link bendy_input_M15_S15: geometry collision mesh filename=../meshes/bendyin.stl scale=1 1 1; visual mesh filename=../meshes/bendyin.stl scale=1 1 1
- link bendy_input_M16_S16: geometry collision mesh filename=../meshes/bendyin.stl scale=1 1 1; visual mesh filename=../meshes/bendyin.stl scale=1 1 1
- link bendy_input_M17_S17: geometry collision mesh filename=../meshes/bendyin.stl scale=1 1 1; visual mesh filename=../meshes/bendyin.stl scale=1 1 1
- link bendy_input_M18_S18: geometry collision mesh filename=../meshes/bendyin.stl scale=1 1 1; visual mesh filename=../meshes/bendyin.stl scale=1 1 1
- link bendy_input_M1_S1: geometry collision mesh filename=../meshes/bendyin.stl scale=1 1 1; visual mesh filename=../meshes/bendyin.stl scale=1 1 1
- link bendy_input_M2_S2: geometry collision mesh filename=../meshes/bendyin.stl scale=1 1 1; visual mesh filename=../meshes/bendyin.stl scale=1 1 1
- link bendy_input_M3_S3: geometry collision mesh filename=../meshes/bendyin.stl scale=1 1 1; visual mesh filename=../meshes/bendyin.stl scale=1 1 1
- link bendy_input_M4_S4: geometry collision mesh filename=../meshes/bendyin.stl scale=1 1 1; visual mesh filename=../meshes/bendyin.stl scale=1 1 1
- link bendy_input_M5_S5: geometry collision mesh filename=../meshes/bendyin.stl scale=1 1 1; visual mesh filename=../meshes/bendyin.stl scale=1 1 1
- link bendy_input_M6_S6: geometry collision mesh filename=../meshes/bendyin.stl scale=1 1 1; visual mesh filename=../meshes/bendyin.stl scale=1 1 1
- link bendy_input_M7_S7: geometry collision mesh filename=../meshes/bendyin.stl scale=1 1 1; visual mesh filename=../meshes/bendyin.stl scale=1 1 1
- link bendy_input_M8_S8: geometry collision mesh filename=../meshes/bendyin.stl scale=1 1 1; visual mesh filename=../meshes/bendyin.stl scale=1 1 1
- link bendy_input_M9_S9: geometry collision mesh filename=../meshes/bendyin.stl scale=1 1 1; visual mesh filename=../meshes/bendyin.stl scale=1 1 1
- link bendy_output_M10_S10: geometry collision mesh filename=../meshes/bendyout.stl scale=1 1 1; visual mesh filename=../meshes/bendyout.stl scale=1 1 1
- link bendy_output_M11_S11: geometry collision mesh filename=../meshes/bendyout.stl scale=1 1 1; visual mesh filename=../meshes/bendyout.stl scale=1 1 1
- link bendy_output_M12_S12: geometry collision mesh filename=../meshes/bendyout.stl scale=1 1 1; visual mesh filename=../meshes/bendyout.stl scale=1 1 1
- link bendy_output_M13_S13: geometry collision mesh filename=../meshes/bendyout.stl scale=1 1 1; visual mesh filename=../meshes/bendyout.stl scale=1 1 1
- link bendy_output_M14_S14: geometry collision mesh filename=../meshes/bendyout.stl scale=1 1 1; visual mesh filename=../meshes/bendyout.stl scale=1 1 1
- link bendy_output_M15_S15: geometry collision mesh filename=../meshes/bendyout.stl scale=1 1 1; visual mesh filename=../meshes/bendyout.stl scale=1 1 1
- link bendy_output_M16_S16: geometry collision mesh filename=../meshes/bendyout.stl scale=1 1 1; visual mesh filename=../meshes/bendyout.stl scale=1 1 1
- link bendy_output_M17_S17: geometry collision mesh filename=../meshes/bendyout.stl scale=1 1 1; visual mesh filename=../meshes/bendyout.stl scale=1 1 1
- link bendy_output_M18_S18: geometry collision mesh filename=../meshes/bendyout.stl scale=1 1 1; visual mesh filename=../meshes/bendyout.stl scale=1 1 1
- link bendy_output_M1_S1: geometry collision mesh filename=../meshes/bendyout.stl scale=1 1 1; visual mesh filename=../meshes/bendyout.stl scale=1 1 1
- link bendy_output_M2_S2: geometry collision mesh filename=../meshes/bendyout.stl scale=1 1 1; visual mesh filename=../meshes/bendyout.stl scale=1 1 1
- link bendy_output_M3_S3: geometry collision mesh filename=../meshes/bendyout.stl scale=1 1 1; visual mesh filename=../meshes/bendyout.stl scale=1 1 1
- link bendy_output_M4_S4: geometry collision mesh filename=../meshes/bendyout.stl scale=1 1 1; visual mesh filename=../meshes/bendyout.stl scale=1 1 1
- link bendy_output_M5_S5: geometry collision mesh filename=../meshes/bendyout.stl scale=1 1 1; visual mesh filename=../meshes/bendyout.stl scale=1 1 1
- link bendy_output_M6_S6: geometry collision mesh filename=../meshes/bendyout.stl scale=1 1 1; visual mesh filename=../meshes/bendyout.stl scale=1 1 1
- link bendy_output_M7_S7: geometry collision mesh filename=../meshes/bendyout.stl scale=1 1 1; visual mesh filename=../meshes/bendyout.stl scale=1 1 1
- link bendy_output_M8_S8: geometry collision mesh filename=../meshes/bendyout.stl scale=1 1 1; visual mesh filename=../meshes/bendyout.stl scale=1 1 1
- link bendy_output_M9_S9: geometry collision mesh filename=../meshes/bendyout.stl scale=1 1 1; visual mesh filename=../meshes/bendyout.stl scale=1 1 1
- link eigenbody_M0_S0: geometry collision mesh filename=../meshes/eigenbody.stl scale=1 1 1; visual mesh filename=../meshes/eigenbody.stl scale=1 1 1
- link foot_input_M25_S25: geometry collision mesh filename=../meshes/foot.stl scale=1 1 1; visual mesh filename=../meshes/foot.stl scale=1 1 1
- link foot_input_M26_S26: geometry collision mesh filename=../meshes/foot.stl scale=1 1 1; visual mesh filename=../meshes/foot.stl scale=1 1 1
- link foot_input_M27_S27: geometry collision mesh filename=../meshes/foot.stl scale=1 1 1; visual mesh filename=../meshes/foot.stl scale=1 1 1
- link foot_input_M28_S28: geometry collision mesh filename=../meshes/foot.stl scale=1 1 1; visual mesh filename=../meshes/foot.stl scale=1 1 1
- link foot_input_M29_S29: geometry collision mesh filename=../meshes/foot.stl scale=1 1 1; visual mesh filename=../meshes/foot.stl scale=1 1 1
- link foot_input_M30_S30: geometry collision mesh filename=../meshes/foot.stl scale=1 1 1; visual mesh filename=../meshes/foot.stl scale=1 1 1
- link static_elbow_M19_S19: geometry collision mesh filename=../meshes/elbow.stl scale=1 1 1; visual mesh filename=../meshes/elbow.stl scale=1 1 1
- link static_elbow_M20_S20: geometry collision mesh filename=../meshes/elbow.stl scale=1 1 1; visual mesh filename=../meshes/elbow.stl scale=1 1 1
- link static_elbow_M21_S21: geometry collision mesh filename=../meshes/elbow.stl scale=1 1 1; visual mesh filename=../meshes/elbow.stl scale=1 1 1
- link static_elbow_M22_S22: geometry collision mesh filename=../meshes/elbow.stl scale=1 1 1; visual mesh filename=../meshes/elbow.stl scale=1 1 1
- link static_elbow_M23_S23: geometry collision mesh filename=../meshes/elbow.stl scale=1 1 1; visual mesh filename=../meshes/elbow.stl scale=1 1 1
- link static_elbow_M24_S24: geometry collision mesh filename=../meshes/elbow.stl scale=1 1 1; visual mesh filename=../meshes/elbow.stl scale=1 1 1
