Commit message: update usd

File: openarm_description/assets/robot/openarm_v1.0/urdf/example/v1.urdf (robot description, URDF)
Before this commit: robot openarm, 26 links, 25 joints
Links:
- removed link openarm_left_hand_tcp
- removed link openarm_right_hand_tcp
- added link openarm_left_ee_tcp
- added link openarm_right_ee_tcp
- link openarm_left_camera_link: geometry collision box size=0.03 0.08 0.03
- link openarm_right_camera_link: geometry collision box size=0.03 0.08 0.03
Joints:
- removed joint openarm_left_hand_tcp_joint
- removed joint openarm_right_hand_tcp_joint
- added joint openarm_left_ee_tcp_joint: type fixed, parent openarm_left_link7, child openarm_left_ee_tcp, origin xyz=0 0 0 rpy=0 0 0
- added joint openarm_right_ee_tcp_joint: type fixed, parent openarm_right_link7, child openarm_right_ee_tcp, origin xyz=0 0 0 rpy=0 0 0
- joint openarm_left_camera_joint: origin xyz=0.0 0.0 0.06 rpy=0 0 0 -> xyz=0.04 0.0 0.0 rpy=0 0 0
- joint openarm_right_camera_joint: origin xyz=0.0 0.0 0.06 rpy=0 0 0 -> xyz=0.04 0.0 0.0 rpy=0 0 0

File: source/isaaclab_assets/data/v1_camera_isaac/urdf/v1_camera.urdf (robot description, URDF)
Before this commit: robot openarm, 26 links, 25 joints
Links:
- removed link openarm_left_hand_tcp
- removed link openarm_right_hand_tcp
- added link openarm_left_ee_tcp
- added link openarm_right_ee_tcp
- link openarm_body_link0: geometry collision mesh filename=package://v1_camera_isaac/mesh/body/collision/body_link0_sy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 scale=0.001 0.001 0.001; visual mesh filename=package://v1_camera_isaac/mesh/body/visual/body_link0.dae scale=0.001 0.001 0.001
- link openarm_left_camera_link: geometry collision box size=0.03 0.08 0.03; visual mesh filename=package://v1_camera_isaac/mesh/arm/visual/cam.dae scale=0.001 -0.001 0.001
- link openarm_left_link0: geometry collision mesh filename=package://v1_camera_isaac/mesh/arm/collision/link0_symp.stl scale=0.001 -0.001 0.001; visual mesh filename=package://v1_camera_isaac/mesh/arm/visual/link0.dae scale=0.001 -0.001 0.001
- link openarm_left_link1: geometry collision mesh filename=package://v1_camera_isaac/mesh/arm/collision/link1_symp.stl scale=0.001 -0.001 0.001; visual mesh filename=package://v1_camera_isaac/mesh/arm/visual/link1.dae scale=0.001 -0.001 0.001
- link openarm_left_link2: geometry collision mesh filename=package://v1_camera_isaac/mesh/arm/collision/link2_symp.stl scale=0.001 -0.001 0.001; visual mesh filename=package://v1_camera_isaac/mesh/arm/visual/link2.dae scale=0.001 -0.001 0.001
- link openarm_left_link3: geometry collision mesh filename=package://v1_camera_isaac/mesh/arm/collision/link3_symp.stl scale=0.001 0.001 0.001; visual mesh filename=package://v1_camera_isaac/mesh/arm/visual/link3.dae scale=0.001 0.001 0.001
- link openarm_left_link4: geometry collision mesh filename=package://v1_camera_isaac/mesh/arm/collision/link4_symp.stl scale=0.001 0.001 0.001; visual mesh filename=package://v1_camera_isaac/mesh/arm/visual/link4.dae scale=0.001 0.001 0.001
- link openarm_left_link5: geometry collision mesh filename=package://v1_camera_isaac/mesh/arm/collision/link5_symp.stl scale=0.001 -0.001 0.001; visual mesh filename=package://v1_camera_isaac/mesh/arm/visual/link5.dae scale=0.001 -0.001 0.001
- link openarm_left_link6: geometry collision mesh filename=package://v1_camera_isaac/mesh/arm/collision/link6_symp.stl scale=0.001 -0.001 0.001; visual mesh filename=package://v1_camera_isaac/mesh/arm/visual/link6.dae scale=0.001 -0.001 0.001
- link openarm_left_link7: geometry collision mesh filename=package://v1_camera_isaac/mesh/arm/collision/link7_symp.stl scale=0.001 -0.001 0.001; visual mesh filename=package://v1_camera_isaac/mesh/arm/visual/link7.dae scale=0.001 -0.001 0.001
- link openarm_right_camera_link: geometry collision box size=0.03 0.08 0.03; visual mesh filename=package://v1_camera_isaac/mesh/arm/visual/cam.dae scale=0.001 0.001 0.001
- link openarm_right_link0: geometry collision mesh filename=package://v1_camera_isaac/mesh/arm/collision/link0_symp.stl scale=0.001 0.001 0.001; visual mesh filename=package://v1_camera_isaac/mesh/arm/visual/link0.dae scale=0.001 0.001 0.001
- link openarm_right_link1: geometry collision mesh filename=package://v1_camera_isaac/mesh/arm/collision/link1_symp.stl scale=0.001 0.001 0.001; visual mesh filename=package://v1_camera_isaac/mesh/arm/visual/link1.dae scale=0.001 0.001 0.001
- link openarm_right_link2: geometry collision mesh filename=package://v1_camera_isaac/mesh/arm/collision/link2_symp.stl scale=0.001 0.001 0.001; visual mesh filename=package://v1_camera_isaac/mesh/arm/visual/link2.dae scale=0.001 0.001 0.001
- link openarm_right_link3: geometry collision mesh filename=package://v1_camera_isaac/mesh/arm/collision/link3_symp.stl scale=0.001 0.001 0.001; visual mesh filename=package://v1_camera_isaac/mesh/arm/visual/link3.dae scale=0.001 0.001 0.001
- link openarm_right_link4: geometry collision mesh filename=package://v1_camera_isaac/mesh/arm/collision/link4_symp.stl scale=0.001 0.001 0.001; visual mesh filename=package://v1_camera_isaac/mesh/arm/visual/link4.dae scale=0.001 0.001 0.001
- link openarm_right_link5: geometry collision mesh filename=package://v1_camera_isaac/mesh/arm/collision/link5_symp.stl scale=0.001 0.001 0.001; visual mesh filename=package://v1_camera_isaac/mesh/arm/visual/link5.dae scale=0.001 0.001 0.001
- link openarm_right_link6: geometry collision mesh filename=package://v1_camera_isaac/mesh/arm/collision/link6_symp.stl scale=0.001 0.001 0.001; visual mesh filename=package://v1_camera_isaac/mesh/arm/visual/link6.dae scale=0.001 0.001 0.001
- link openarm_right_link7: geometry collision mesh filename=package://v1_camera_isaac/mesh/arm/collision/link7_symp.stl scale=0.001 0.001 0.001; visual mesh filename=package://v1_camera_isaac/mesh/arm/visual/link7.dae scale=0.001 0.001 0.001
Joints:
- removed joint openarm_left_hand_tcp_joint
- removed joint openarm_right_hand_tcp_joint
- added joint openarm_left_ee_tcp_joint: type fixed, parent openarm_left_link7, child openarm_left_ee_tcp, origin xyz=0 0 0 rpy=0 0 0
- added joint openarm_right_ee_tcp_joint: type fixed, parent openarm_right_link7, child openarm_right_ee_tcp, origin xyz=0 0 0 rpy=0 0 0
- joint openarm_left_camera_joint: origin xyz=0.04 0.0 0.0 rpy=0 0 0 -> xyz=0.0 0.0 0.06 rpy=0 0 0
- joint openarm_right_camera_joint: origin xyz=0.04 0.0 0.0 rpy=0 0 0 -> xyz=0.0 0.0 0.06 rpy=0 0 0
